Commit message: First more less working gazebo model of justina

File: catkin_ws/src/hardware/justina_description/urdf/justina.urdf (robot description, URDF)
Before this commit: robot justina, 36 links, 35 joints
Joints:
- removed joint pan_connect
- removed joint tilt_connect
- added joint head_pan: type revolute, parent head_link1, child head_link2, origin xyz=0.0 0 0.05 rpy=0 0 0, axis 0 0 1, limit lower=-3.14 upper=3.14 effort=6.0 velocity=3.0
- added joint head_tilt: type revolute, parent head_link2, child neck_link, origin xyz=0.0 0 0.06 rpy=0 0 0, axis 0 -1 0, limit lower=-1.2 upper=1.0 effort=6.0 velocity=3.0
- joint la_1_joint: limit lower=-1.7 upper=1.7 effort=1000 velocity=10 -> lower=-1.7 upper=1.7 effort=16.0 velocity=3.0
- joint la_2_joint: limit lower=-0.75 upper=1.85 effort=1000 velocity=10 -> lower=-0.75 upper=1.85 effort=8.0 velocity=3.0
- joint la_3_joint: limit lower=-2.5 upper=2.5 effort=1000 velocity=10 -> lower=-2.5 upper=2.5 effort=6.0 velocity=3.0
- joint la_4_joint: limit lower=-1.8 upper=1.8 effort=1000 velocity=10 -> lower=-1.8 upper=1.8 effort=8.0 velocity=3.0
- joint la_5_joint: limit lower=-2.5 upper=2.5 effort=1000 velocity=10 -> lower=-2.5 upper=2.5 effort=6.0 velocity=3.0
- joint la_6_joint: limit lower=-1.4 upper=1.57 effort=1000 velocity=10 -> lower=-1.4 upper=1.57 effort=6.0 velocity=3.0
- joint la_7_joint: limit lower=-2.5 upper=2.5 effort=1000 velocity=10 -> lower=-2.5 upper=2.5 effort=3.0 velocity=3.0
- joint la_grip_left: limit lower=-0.3 upper=1.5 effort=1000 velocity=10 -> lower=-0.3 upper=1.5 effort=3.0 velocity=3.0
- joint la_grip_right: limit lower=-0.3 upper=1.5 effort=1000 velocity=10 -> lower=-0.3 upper=1.5 effort=3.0 velocity=3.0
- joint ra_1_joint: limit lower=-1.7 upper=1.7 effort=1000 velocity=10 -> lower=-1.7 upper=1.7 effort=16.0 velocity=3.0
- joint ra_2_joint: limit lower=-1.85 upper=0.75 effort=1000 velocity=10 -> lower=-1.85 upper=0.75 effort=8.0 velocity=3.0
- joint ra_3_joint: limit lower=-2.5 upper=2.5 effort=1000 velocity=10 -> lower=-2.5 upper=2.5 effort=6.0 velocity=3.0
- joint ra_4_joint: limit lower=-1.8 upper=1.8 effort=1000 velocity=10 -> lower=-1.8 upper=1.8 effort=8.0 velocity=3.0
- joint ra_5_joint: limit lower=-2.5 upper=2.5 effort=1000 velocity=10 -> lower=-2.5 upper=2.5 effort=6.0 velocity=3.0
- joint ra_6_joint: limit lower=-1.4 upper=1.57 effort=1000 velocity=10 -> lower=-1.4 upper=1.57 effort=6.0 velocity=3.0
- joint ra_7_joint: limit lower=-2.5 upper=2.5 effort=1000 velocity=10 -> lower=-2.5 upper=2.5 effort=3.0 velocity=3.0
- joint ra_grip_left: limit lower=-0.3 upper=1.5 effort=1000 velocity=10 -> lower=-0.3 upper=1.5 effort=3.0 velocity=3.0
- joint ra_grip_right: limit lower=-0.3 upper=1.5 effort=1000 velocity=10 -> lower=-0.3 upper=1.5 effort=3.0 velocity=3.0
