Commit message: Some updates to justina description

File: catkin_ws/src/hardware/justina_description/urdf/test_base.xacro (robot description, xacro)
@@ -2,172 +2,291 @@
 <robot name="justina" xmlns:xacro="http://www.ros.org/wiki/xacro">
   <!-- INCLUDES -->
-    <xacro:include filename="$(find justina_description)/urdf/test_parameters.xacro" />
-    <!-- BASE LINK -->
-    <link name="base_link">
-        <material name="orange"/>
-        <!-- pose and inertial -->
-        <pose>0 0 0 0 0 0</pose>
-        <inertial>
-            <origin rpy="0 0 0" xyz="${-base_size_x/2 + wheel_radius} 0 ${wheel_radius/2}"/>
-            <mass value="${base_mass}"/>
-            <xacro:box_inertia mass="${base_mass}" x="${base_size_x}" y="${base_size_y}" z="${base_size_z}"/>
-        </inertial>
-        <!-- body -->
-        <collision name="base_front_collision">
-            <origin rpy="0 0 0" xyz="${-base_size_x/2 + wheel_radius} 0 ${wheel_radius/2}"/>
-            <geometry>
-                <box size="${base_size_x} ${base_size_y} ${base_size_z}"/>
-            </geometry>
-        </collision>
-        <visual>
-            <origin rpy="0 0 0" xyz="${-base_size_x/2 + wheel_radius} 0 ${wheel_radius/2}"/>
-            <geometry>
-                <box size="${base_size_x} ${base_size_y} ${base_size_z}"/>
-            </geometry>
-            <material name="green"/>
-        </visual>
-        <!-- caster rear -->
-        <collision name="caster_front_collision">
-            <origin rpy=" 0 0 0" xyz="-${base_size_x-wheel_radius-wheel_radius/4} 0 ${-wheel_radius/2}"/>
-            <geometry>
-                <sphere radius="${wheel_radius/2}"/>
-            </geometry>
-        </collision>
-        <visual>
-            <origin rpy=" 0 0 0" xyz="-${base_size_x-wheel_radius-wheel_radius/4} 0 ${-wheel_radius/2}"/>
-            <geometry>
-                <sphere radius="${wheel_radius/2}"/>
-            </geometry>
-            <material name="gray"/>
-        </visual>
-    </link>
-    <!-- LEFT WHEEL LINK -->
-    <link name="left_wheel_link">
-        <inertial>
-            <mass value="${wheel_mass}"/>
-            <origin rpy="0 1.5707 1.5707" xyz="0 0 0"/>
-            <xacro:cylinder_inertia mass="${wheel_mass}" r="${wheel_radius}" l="${wheel_width}"/>
-        </inertial>
-        <collision name="left_wheel_collision">
-            <origin rpy="0 1.5707 1.5707" xyz="0 0 0"/>
-            <geometry>
-                <cylinder radius="${wheel_radius}" length="${wheel_width}"/>
-            </geometry>
-        </collision>
-        <visual>
-            <origin rpy="0 1.5707 1.5707" xyz="0 0 0"/>
-            <geometry>
-                <cylinder radius="${wheel_radius}" length="${wheel_width}"/>
-            </geometry>
-            <material name="gray"/>
-        </visual>
-    </link>
-    <!-- LEFT WHEEL JOINT -->
-    <joint name="left_motor" type="continuous">
-        <origin rpy="0 0 0" xyz="0.0 ${base_size_y/2+wheel_width/2} 0.0"/>
-        <child link="left_wheel_link"/>
-        <parent link="base_link"/>
-        <axis rpy="0 0 0" xyz="0 1 0"/>
-        <dynamics damping="${motor_damping}" friction="${motor_friction}"/>
-    </joint>
-    <!-- RIGHT WHEEL LINK -->
-    <link name="right_wheel_link">
-        <inertial>
-            <mass value="${wheel_mass}"/>
-            <origin rpy="0 1.5707 1.5707" xyz="0 0 0"/>
-            <xacro:cylinder_inertia mass="${wheel_mass}" r="${wheel_radius}" l="${wheel_width}"/>
-        </inertial>
-        <collision name="right_wheel_collision">
-            <origin rpy="0 1.5707 1.5707" xyz="0 0 0"/>
-            <geometry>
-                <cylinder radius="${wheel_radius}" length="${wheel_width}"/>
-            </geometry>
-        </collision>
-        <visual>
-            <origin rpy="0 1.5707 1.5707" xyz="0 0 0"/>
-            <geometry>
-                <cylinder radius="${wheel_radius}" length="${wheel_width}"/>
-            </geometry>
-            <material name="gray"/>
-        </visual>
-    </link>
-    <!-- RIGHT WHEEL JOINT -->
-    <joint name="right_motor" type="continuous">
-        <origin rpy="0 0 0" xyz="0 ${-base_size_y/2-wheel_width/2} 0"/>
-        <child link="right_wheel_link"/>
-        <parent link="base_link"/>
-        <axis rpy="0 0 0" xyz="0 1 0"/>
-        <dynamics damping="${motor_damping}" friction="${motor_friction}"/>
-    </joint>
-    <!-- TRANSMISSIONS -->
-    <transmission name="left_motor_transmission">
-        <type>transmission_interface/SimpleTransmission</type>
-        <joint name="left_motor">
-            <hardwareInterface>hardware_interface/EffortJointInterface</hardwareInterface>
-        </joint>
-        <actuator name="left_motor">
-            <hardwareInterface>hardware_interface/EffortJointInterface</hardwareInterface>
-            <mechanicalReduction>1</mechanicalReduction>
-        </actuator>
-    </transmission>
-    <transmission name="right_motor_transmission">
-        <type>transmission_interface/SimpleTransmission</type>
-        <joint name="right_motor">
-            <hardwareInterface>hardware_interface/EffortJointInterface</hardwareInterface>
-        </joint>
-        <actuator name="right_motor">
-            <hardwareInterface>hardware_interface/EffortJointInterface</hardwareInterface>
-            <mechanicalReduction>1</mechanicalReduction>
-        </actuator>
-    </transmission>
-    <gazebo reference="left_wheel_link">
-      <mu1 value="100.0" />
-      <mu2 value="100.0" />
-      <kp  value="1000000.0" />
-      <kd  value="1.0" />
-      <maxVel  value="100.0" />
-      <minDepth  value="0.0" />
-    </gazebo>
-    <gazebo reference="right_wheel_link">
-      <mu1 value="100.0" />
-      <mu2 value="100.0" />
-      <kp  value="1000000.0" />
-      <kd  value="1.0" />
-      <maxVel  value="100.0" />
-      <minDepth  value="0.0" />
-    </gazebo>
-    <gazebo reference="base_link">
-      <mu1 value="0.0" />
-      <mu2 value="0.0" />
-      <kp  value="1000000.0" />
-      <kd  value="1.0" />
-    </gazebo>
+  <xacro:property name="base_width" value="0.42"/>
+  <xacro:property name="base_depth" value="0.42"/>
+  <xacro:property name="base_height" value="0.2"/>
+  <xacro:property name="base_mass" value="30.0"/>
+  <xacro:property name="wheel_radius" value="0.06"/>
+  <xacro:property name="wheel_height" value="0.04"/>
+  <xacro:property name="wheel_mass" value="30.0"/>
+  <xacro:property name="torso_mass" value="0.6"/>
+  <xacro:property name="spine_mass" value="0.001"/>
+  <xacro:property name="neck_mass" value="0.001"/>
+  <xacro:property name="MX_106_mass" value="0.05"/>
+  <xacro:property name="MX_64_mass" value="0.05"/>
+  <xacro:property name="kinect_mass" value="0.1"/>
+  <xacro:property name="PI_2" value="1.570796327"/>
+  <xacro:property name="PI" value="3.14159265359"/>
+  <!-- BASE LINK -->
+  <link name="base_link">
+    <visual>
+      <origin xyz="0 0 0.235" rpy="0 0 0"/>
+      <geometry> <box size="0.42 0.42 0.2"/></geometry>
+      <material name="blue"/>
+    </visual>
+    <collision>
+      <origin xyz="0 0 0.235" rpy="0 0 0"/>
+      <geometry> <box size="0.42 0.42 0.2"/></geometry>
+    </collision>
+    <inertial>
+      <origin xyz="0 0 0.235" rpy="0 0 0"/>
+      <mass value="50.00"/>
+      <!--<box_inertia m="${base_mass}" x="0.42" y="0.42" z="0.2"/>-->
+      <inertia ixx="0.3742" ixy="0.000434172172" ixz="0.03088" iyy="0.3436" iyz="0.01775" izz="0.1509"/>
+    </inertial>
+  </link>
+  <joint name="wheel_left_connect" type="continuous">
+    <origin xyz="0 0.24 0.065" rpy="-1.5708 0 0"/>
+    <!--<origin rpy="0.0 0.0 0.0" xyz="-0.11 0.133 0.04"/>-->
+    <parent link="base_link"/>
+    <child link="wheel_left"/>
+    <axis xyz="0.0 0 1.0"/>
+    <limit effort="11.067" velocity="20.8"/>
+    <dynamics damping="1.0"/>
+  </joint>
+  <link name="wheel_left">
+    <visual>
+      <!--<origin rpy="1.57079632679 0.0 0.0" xyz="0.0 0.0 0.0"/>-->
+      <origin xyz="0 0 0" rpy="0 0 0"/>
+      <geometry><cylinder length="${wheel_height}" radius="${wheel_radius}"/></geometry>
+      <material name="gray"><color rgba="0 0 0 1" /></material>
+    </visual>
+    <collision>
+      <!--<origin rpy="1.57079632679 0.0 0.0" xyz="0.0 0.0 0.0"/>-->
+      <origin xyz="0 0 0" rpy="0 0 0"/>
+	<geometry><cylinder length="${wheel_height}" radius="${wheel_radius}"/></geometry>
+    </collision>
+    <inertial>
+      <origin xyz="0 0 0"/>
+      <mass value="0.2"/>
+      <inertia ixx="0.015" ixy="0" ixz="0" iyy="0.015" iyz="0" izz="0.015"/>
+    </inertial>
+  </link>
+  <joint name="wheel_right_connect" type="continuous">
+    <origin xyz="0 -0.24 0.065" rpy="-1.5708 0 0"/>
+    <!--<origin rpy="0.0 0.0 0.0" xyz="-0.11 -0.133 0.04"/>-->
+    <parent link="base_link"/>
+    <child link="wheel_right"/>
+    <axis xyz="0.0 0 1.0"/>
+    <limit effort="11.067" velocity="20.8"/>
+    <dynamics damping="1.0"/>
+  </joint>
+  <link name="wheel_right">
+    <visual>
+      <!--<origin rpy="1.57079632679 0.0 0.0" xyz="0.0 0.0 0.0"/>-->
+      <origin xyz="0 0 0" rpy="0 0 0"/>
+      <geometry><cylinder length="${wheel_height}" radius="${wheel_radius}"/></geometry>
+      <material name="black"><color rgba="0 0 0 1" /></material>
+    </visual>
+    <collision>
+      <!--<origin rpy="1.57079632679 0.0 0.0" xyz="0.0 0.0 0.0"/>-->
+      <origin xyz="0 0 0" rpy="0 0 0"/>
+      <geometry><cylinder length="${wheel_height}" radius="${wheel_radius}"/></geometry>
+    </collision>
+    <inertial>
+      <origin xyz="0 0 0" rpy="0 0 0"/>
+      <mass value="0.2"/>
+      <inertia ixx="0.015" ixy="0" ixz="0" iyy="0.015" iyz="0" izz="0.015"/>
+    </inertial>
+  </link>
+  <joint name="wheel_back_connect_x" type="continuous">
+    <!--<origin rpy="0.0 0.0 0.0" xyz="0.1495                 -0.055                 0.03"/>-->
+    <origin xyz="-0.24 0 0.065" rpy="-1.5708 0 -1.5708"/>
+    <parent link="base_link"/>
+    <child link="wheel_back_x"/>
+    <axis xyz="1 0 0"/>
+    <limit effort="1.0" velocity="3.0"/>
+    <dynamics damping="1.0"/>
+  </joint>
+  <link name="wheel_back_x">
+    <inertial>
+      <origin xyz="0 0 0" rpy="0 0 0"/>
+      <mass value="0.2"/>
+      <inertia ixx="0.015" ixy="0" ixz="0" iyy="0.015" iyz="0" izz="0.015"/>
+    </inertial>
+  </link>
+  <joint name="wheel_back_connect_y" type="continuous">
+    <axis xyz="0 1 0"/>
+    <limit effort="8.85" velocity="10.0"/>
+    <parent link="wheel_back_x"/>
+    <child link="wheel_back_y"/>
+  </joint>
+  <link name="wheel_back_y">
+    <inertial>
+      <mass value="0.2"/>
+      <origin xyz="0 0 0"/>
+      <inertia ixx="0.015" ixy="0" ixz="0" iyy="0.015" iyz="0" izz="0.015"/>
+    </inertial>
+  </link>
+  <joint name="wheel_back_connect_z" type="continuous">
+      <axis xyz="0.0 0.0 1.0"/>
+      <limit effort="8.85" velocity="10.0"/>
+      <parent link="wheel_back_y"/>
+      <child link="wheel_back_z"/>
+  </joint>
+  <link name="wheel_back_z">
+    <visual>
+      <geometry>
+        <sphere radius="0.06"/>
+      </geometry>
+      <material name="wheel"/>
+    </visual>
+    <collision>
+      <geometry>
+        <sphere radius="0.06"/>
+      </geometry>
+    </collision>
+    <inertial>
+      <mass value="0.2"/>
+      <origin xyz="0 0 0"/>
+      <inertia ixx="0.015" ixy="0" ixz="0" iyy="0.015" iyz="0" izz="0.015"/>
+    </inertial>
+  </link>
+	<joint name="wheel_front_connect_x" type="continuous">
+		<!--<origin rpy="0.0 0.0 0.0" xyz="0.1495                 0.055                 0.03"/>-->
+		<origin xyz="0.24 0 0.065" rpy="-1.5708 0 -1.5708"/>
+		<parent link="base_link"/>
+		<child link="wheel_front_x"/>
+		<axis xyz="1 0 0"/>
+    		<limit effort="1.0" velocity="3.0"/>
+    		<dynamics damping="1.0"/>
+	</joint>
+  <link name="wheel_front_x">
+    <inertial>
+      <mass value="0.2"/>
+      <origin xyz="0 0 0"/>
+      <inertia ixx="0.015" ixy="0" ixz="0" iyy="0.015" iyz="0" izz="0.015"/>
+    </inertial>
+  </link>
+  <joint name="wheel_front_connect_y" type="continuous">
+    <axis xyz="0.0 1.0 0.0"/>
+    <limit effort="8.85" velocity="10.0"/>
+    <parent link="wheel_front_x"/>
+    <child link="wheel_front_y"/>
+  </joint>
+  <link name="wheel_front_y">
+    <inertial>
+      <mass value="0.2"/>
+      <origin xyz="0 0 0"/>
+      <inertia ixx="0.015" ixy="0" ixz="0" iyy="0.015" iyz="0" izz="0.015"/>
+    </inertial>
+  </link>
+  <joint name="wheel_front_connect_z" type="continuous">
+    <axis xyz="0.0 0.0 1.0"/>
+    <limit effort="8.85" velocity="10.0"/>
+    <parent link="wheel_front_y"/>
+    <child link="wheel_front_z"/>
+  </joint>
+  <link name="wheel_front_z">
+    <visual>
+      <geometry>
+        <sphere radius="0.06"/>
+      </geometry>
+      <material name="wheel"/>
+    </visual>
+    <collision>
+      <geometry>
+        <sphere radius="0.06"/>
+      </geometry>
+    </collision>
+    <inertial>
+      <mass value="0.2"/>
+      <origin xyz="0 0 0"/>
+      <inertia ixx="0.015" ixy="0" ixz="0" iyy="0.015" iyz="0" izz="0.015"/>
+    </inertial>
+  </link>
+  	<gazebo reference="base_link">
+		<material>Gazebo/blue</material>
+    <selfCollide>false</selfCollide>
+    <gravity>true</gravity>
+    <mu1>0.9</mu1>
+    <mu2>0.9</mu2>
+	</gazebo>
+	<gazebo reference="wheel_left">
+		<material>Gazebo/Black</material>
+		    <selfCollide>false</selfCollide>
+		    <gravity>true</gravity>
+		    <turnGravityOff>false</turnGravityOff>
+		    <kp>1000000.0</kp>
+		    <kd>10.0</kd>
+		    <mu1>1.0</mu1>
+		    <mu2>1.0</mu2>
+		    <fdir1>1 0 0</fdir1>
+		    <maxVel>1.0</maxVel>
+		    <minDepth>0.00</minDepth>
+	</gazebo>
+	<gazebo reference="wheel_right">
+		<material>Gazebo/Black</material>
+    <selfCollide>false</selfCollide>
+    <gravity>true</gravity>
+    <turnGravityOff>false</turnGravityOff>
+    <kp>1000000.0</kp>
+    <kd>10.0</kd>
+    <mu1>1.0</mu1>
+    <mu2>1.0</mu2>
+    <fdir1>1 0 0</fdir1>
+    <maxVel>1.0</maxVel>
+    <minDepth>0.00</minDepth>
+	</gazebo>
+  <gazebo reference="wheel_back_y">
+    <selfCollide>false</selfCollide>
+    <gravity>true</gravity>
+    <mu1>0.1</mu1>
+    <mu2>0.1</mu2>
+    <maxVel>1.0</maxVel>
+    <material value="Gazebo/FlatBlack"/>
+  </gazebo>
+  <gazebo reference="wheel_front_z">
+    <selfCollide>false</selfCollide>
+    <gravity>true</gravity>
+    <mu1>0.1</mu1>
+    <mu2>0.1</mu2>
+    <maxVel>1.0</maxVel>
+    <material value="Gazebo/FlatBlack"/>
+  </gazebo>
+  <transmission name="tran1">
+	    <type>transmission_interface/SimpleTransmission</type>
+	    <joint name="wheel_left_connect">
+		    <hardwareInterface>hardware_interface/EffortJointInterface</hardwareInterface>
+	    </joint>
+	    <actuator name="motor1">
+		    <mechanicalReduction>1</mechanicalReduction>
+	    </actuator>
+    </transmission>
+    <transmission name="tran2">
+	    <type>transmission_interface/SimpleTransmission</type>
+	    <joint name="wheel_right_connect">
+		    <hardwareInterface>hardware_interface/EffortJointInterface</hardwareInterface>
+	    </joint>
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