Commit message: Add nodes for webcam_man and kinect_man. Modify web_cam to publish only one topic Change speed check in omni_base_node and change also tick calculation from metric speeds Add maps and prohibition maps for biorobotics lab Add and change launch to launch separately base, upper actuators and cameras

File: catkin_ws/src/hardware/justina_description/urdf/justina_base.xacro (robot description, xacro)
@@ -189,8 +189,29 @@
     </inertial>
   </link>
+  <link name="laser_link_rear">
+    <visual>
+      <origin xyz="0 0 0" rpy="0 0 0"/>
+      <geometry> <box size="0.08 0.08 0.1"/></geometry>
+      <material name="black"/>
+    </visual>
+    <collision>
+      <origin xyz="0 0 0" rpy="0 0 0"/>
+      <geometry> <box size="0.08 0.08 0.1"/></geometry>
+    </collision>
+    <inertial>
+      <origin xyz="0 0 0" rpy="0 0 0"/>
+      <mass value="0.1"/>
+      <xacro:box_inertia m="${0.05}" x="${0.08}" y="${0.08}" z="${0.1}"/>
+    </inertial>
+  </link>
   <joint name="laser_connect" type="fixed">
-    <origin xyz="0.1 0 0.44" />
+    <origin xyz="0.17 0 0.44" />
     <parent link="base_link"/>
     <child link="laser_link"/>
   </joint>
+  <joint name="rear_laser_connect" type="fixed">
+    <origin xyz="-0.2 0 0.41" rpy="0 0 ${PI}"/>
+    <parent link="base_link"/>
+    <child link="laser_link_rear"/>
+  </joint>
 </robot>
