Commit message: Correct urdf and justina_controllers to make torso ready Modify topic_resender.py node to publish current head and arms positions Copy obj_reco node from justina repo and modify GUI to call find_lines service

File: catkin_ws/src/hardware/justina_description/urdf/justina_torso.xacro (robot description, xacro)
@@ -30,5 +30,6 @@
     <parent link="torso_link"/>
     <child link="spine_link"/>
-    <limit effort="1000" lower="0.2" upper="0.5" velocity="0.2"/>
+    <limit effort="1000" lower="0.0" upper="0.5" velocity="0.2"/>
+    <dynamics damping ="0.1" />
     <axis xyz="0 0 1" />
   </joint>
