Commit message: Correct head limits in justina_head.xacro Correct inverse kinematics to use the new srv ForwardKinematics Small style changes in navigation nodes Add node to translate topics from gazebo controllers to justina-like topics

File: catkin_ws/src/hardware/justina_description/urdf/justina_head.xacro (robot description, xacro)
@@ -45,5 +45,5 @@
     <axis xyz="0 0 1" />
     <dynamics damping ="0.1" />
-    <limit effort="6.0" velocity="3.0" lower="-3.14" upper="3.14"/>
+    <limit effort="6.0" velocity="3.0" lower="-1.57" upper="1.57"/>
   </joint>
   <link name="neck_link">

Commit message: Change justina_head description to include the realsense camera_link frame Change cloud topic in rviz

File: catkin_ws/src/hardware/justina_description/urdf/justina_head.xacro (robot description, xacro)
@@ -75,34 +75,34 @@
     <limit effort="6.0" velocity="3.0" lower="-1.2" upper="1.0"/>
   </joint>
-  <link name="kinect_base">
+  <link name="camera_link">
     <visual>
       <origin xyz="0 0 0" rpy="0 0 0"/>
       <geometry>
-        <box size=" 0.058 0.207 0.04"/>
+        <box size=" 0.029 0.103 0.02"/>
       </geometry>
-      <material name="black"/>
+      <material name="gray"/>
     </visual>
     <collision>
       <origin xyz= "0 0 0" rpy="0 0 0"/>
       <geometry>
-        <box size=" 0.058 0.207 0.04"/>
+        <box size=" 0.029 0.103 0.02"/>
       </geometry>
     </collision>
     <inertial>
       <origin xyz="0.0 0 0.0" rpy = "0 0 0"/>
-      <mass value = "0.15" />
+      <mass value = "0.1" />
       <inertia ixx = "0.00006205" iyy = "0.000555" izz = "0.0005776" ixy = "0" ixz = "0" iyz = "0" />
     </inertial>
   </link>
-  <joint name="kinect_base_connect" type="fixed">
+  <joint name="camera_link_connect" type="fixed">
     <origin xyz="0 0 0.065" rpy="0 0 0"/>
     <parent link="neck_link"/>
-    <child link="kinect_base"/>
+    <child link="camera_link"/>
   </joint>
-  <link name="kinect_link"/>
+  <!--link name="kinect_link"/>
   <joint name="kinect_connect" type="fixed">
     <origin xyz="0 0 0" rpy="-1.5708 0 -1.5708"/>
     <parent link="kinect_base"/>
     <child link="kinect_link"/>
-  </joint>
+  </joint-->
 </robot>

Commit message: Add line to install gmapping to Setup.sh Create new node for head using similar program to arm_node Add trajectory subscriber to arm node Remove hardware_tools dependence in head Correct servo limits in head servos Create new head_params.yaml file for the new head_node Remove tilt_bias in justina_head.xacro. Now is set to zero. Change GUI to allow wider pan-tilt ranges. Create new biorobotics map and modify launches to use new head node and realsense for navigation

File: catkin_ws/src/hardware/justina_description/urdf/justina_head.xacro (robot description, xacro)
@@ -68,5 +68,5 @@
   </link>
   <joint name="head_tilt" type="revolute">
-    <origin xyz="0.0 0 0.06" rpy="0 -0.08 0"/>
+    <origin xyz="0.0 0 0.06" rpy="0 0 0"/>
     <parent link="head_link2"/>
     <child link="neck_link"/>
