Commit message: Correct sizes and joint origins in justina.xacro and justina_head.xacro to correct physical error positions Correct kinect man node to publish point clouds with stamps Correct parameters in justina navigation launch files

File: catkin_ws/src/hardware/justina_description/urdf/justina.xacro (robot description, xacro)
@@ -9,5 +9,5 @@
   <xacro:include filename="$(find justina_description)/urdf/justina_head.xacro"/>
   <joint name="torso_connect" type="fixed">
-    <origin xyz= "0 0 0.9" rpy="0 0 0"/>
+    <origin xyz= "0 0 1.08" rpy="0 0 0"/>
     <parent link="base_link"/>
     <child link="torso_link"/>

File: catkin_ws/src/hardware/justina_description/urdf/justina_head.xacro (robot description, xacro)
@@ -68,5 +68,5 @@
   </link>
   <joint name="head_tilt" type="revolute">
-    <origin xyz="0.0 0 0.06" rpy="0 0 0" />
+    <origin xyz="0.0 0 0.06" rpy="0 -0.08 0"/>
     <parent link="head_link2"/>
     <child link="neck_link"/>

Commit message: Correct servo zero params add new biorobotics map correct torso position in urdf correct launch files

File: catkin_ws/src/hardware/justina_description/urdf/justina.xacro (robot description, xacro)
@@ -9,5 +9,5 @@
   <xacro:include filename="$(find justina_description)/urdf/justina_head.xacro"/>
   <joint name="torso_connect" type="fixed">
-    <origin xyz= "0 0 1.08" rpy="0 0 0"/>
+    <origin xyz= "0.05 0 1.08" rpy="0 0 0"/>
     <parent link="base_link"/>
     <child link="torso_link"/>

Commit message: Delete unused files for omni base simulation in gazebo Add new justina_base_omni files for omni base simulation Add node for omni base control and odometry calculation Correct the corresponding launch files

File: catkin_ws/src/hardware/justina_description/urdf/justina.xacro (robot description, xacro)
@@ -3,5 +3,5 @@
   <xacro:include filename="$(find justina_description)/urdf/macros.xacro"/>
   <xacro:include filename="$(find justina_description)/urdf/materials.xacro"/>
-  <xacro:include filename="$(find justina_description)/urdf/justina_base.xacro"/>
+  <xacro:include filename="$(find justina_description)/urdf/justina_base_omni.xacro"/>
   <xacro:include filename="$(find justina_description)/urdf/justina_torso.xacro"/>
   <xacro:include filename="$(find justina_description)/urdf/justina_left_arm.xacro"/>

File: catkin_ws/src/hardware/justina_description/urdf/justina_base_omni.xacro (robot description, xacro)
@@ -1,12 +1,14 @@
 <?xml version="1.0"?>
 <robot name="justina" xmlns:xacro="http://www.ros.org/wiki/xacro">
-  <xacro:property name="base_radius" value="0.2"/>
+  <xacro:property name="base_radius" value="0.21"/>
   <xacro:property name="base_height" value="0.2"/>
-  <xacro:property name="base_mass"   value="10.0"/>
+  <xacro:property name="base_mass"   value="20.0"/>
   <xacro:property name="wheel_radius" value="0.08"/>
-  <xacro:property name="wheel_width"  value="0.03"/>
+  <xacro:property name="wheel_width"  value="0.01"/>
   <xacro:property name="wheel_mass"   value="0.5"/>
   <xacro:property name="PI" value="3.14159265358979323846"/>
-  <xacro:include filename="$(find justina_description)/urdf/justina_base_rim.xacro"/>
+  <xacro:include filename="$(find justina_description)/urdf/macros.xacro"/>
+  <xacro:include filename="$(find justina_description)/urdf/justina_base_omni.gazebo"/>
+  <!-- MAIN BASE LINK -->
   <link name="base_link"/>
   <link name="base_center">
@@ -24,4 +26,19 @@
     </collision>
   </link>
+  <link name="base_torso_support">
+    <inertial>
+      <origin xyz="0 0 0"/>
+      <mass value="0.5"/>
+      <xacro:box_inertia m="0.5" x="0.12" y="0.12" z="0.16"/>
+    </inertial>
+    <visual>
+      <origin xyz="0 0 0" rpy="0 0 0"/>
+      <geometry> <box size="0.12 0.12 0.16"/></geometry>
+      <material name="black"/>
+    </visual>
+    <collision>
+      <geometry> <box size="0.12 0.12 0.16"/></geometry>
+    </collision>
+  </link>
   <joint name="base_joint" type="fixed">
     <parent link="base_link" />
@@ -29,9 +46,9 @@
     <origin xyz="0 0 0.1905"/>
   </joint>
-  <gazebo reference="base_center">
-    <material>Gazebo/Blue</material>
-    <selfCollide>false</selfCollide>
-    <gravity>true</gravity>
-  </gazebo>
+  <joint name="base_torso_support_joint" type="fixed">
+    <parent link="base_center" />
+    <child link="base_torso_support" />
+    <origin xyz="0 0 0.18"/>
+  </joint>
   <!-- LEFT WHEEL ACTUATOR-->
   <link name="left_wheel_link">
@@ -54,30 +71,7 @@
     <axis xyz="0 0 1"/>
     <origin xyz="${(base_radius+0.03)*cos( PI/3)} ${(base_radius+0.03)*sin( PI/3)} -0.05" rpy="${PI/2} 0 ${ PI/3+PI/2}"/>
-    <limit velocity="30.0" effort="0.6"/>
+    <limit velocity="30.0" effort="1.0"/>
+    <dynamics damping="1.0" friction="0.01"/>
   </joint>
-  <transmission name="wheel_left_transmission">
-    <type>transmission_interface/SimpleTransmission</type>
-    <joint name="wheel_left_joint">
-      <hardwareInterface>hardware_interface/EffortJointInterface</hardwareInterface>
-    </joint>
-    <actuator name="wheel_left_motor">
-      <hardwareInterface>hardware_interface/EffortJointInterface</hardwareInterface>
-      <mechanicalReduction>1</mechanicalReduction>
-    </actuator>
-  </transmission>
-  <gazebo reference="left_wheel_link">
-    <material>Gazebo/Black</material>
-    <selfCollide>false</selfCollide>
-    <gravity>true</gravity>
-    <collision name="left_wheel_link_collision">
-      <surface><friction>
-        <ode>
-          <mu>0.1</mu>
-          <mu2>15</mu2>
-          <fdir1>0 0 1</fdir1>
-        </ode></friction>
-      </surface>
-    </collision>
-  </gazebo>
   <!-- RIGHT WHEEL ACTUATOR-->
   <link name="right_wheel_link">
@@ -100,30 +94,7 @@
     <axis xyz="0 0 1"/>
     <origin xyz="${(base_radius+0.03)*cos(-PI/3)} ${(base_radius+0.03)*sin(-PI/3)} -0.05" rpy="${PI/2} 0 ${-PI/3+PI/2}"/>
-    <limit velocity="30.0" effort="0.6"/>
+    <limit velocity="30.0" effort="1.0"/>
+    <dynamics damping="1.0" friction="0.01"/>
   </joint>
-  <transmission name="wheel_right_transmission">
-    <type>transmission_interface/SimpleTransmission</type>
-    <joint name="wheel_right_joint">
-      <hardwareInterface>hardware_interface/EffortJointInterface</hardwareInterface>
-    </joint>
-    <actuator name="wheel_right_motor">
-      <hardwareInterface>hardware_interface/EffortJointInterface</hardwareInterface>
-      <mechanicalReduction>1</mechanicalReduction>
-    </actuator>
-  </transmission>
-  <gazebo reference="right_wheel_link">
-    <material>Gazebo/Black</material>
-    <selfCollide>false</selfCollide>
-    <gravity>true</gravity>
-    <collision name="right_wheel_link_collision">
-      <surface><friction>
-        <ode>
-          <mu>0.1</mu>
-          <mu2>15</mu2>
-          <fdir1>0 0 1</fdir1>
-        </ode></friction>
-      </surface>
-    </collision>
-  </gazebo>
   <!-- BACK WHEEL ACTUATOR-->
   <link name="back_wheel_link">
@@ -146,29 +117,49 @@
     <axis xyz="0 0 1"/>
     <origin xyz="${(base_radius+0.03)*cos(PI)} ${(base_radius+0.03)*sin(PI)} -0.05" rpy="${PI/2} 0 ${PI+PI/2}"/>
-    <limit velocity="30.0" effort="0.6"/>
+    <limit velocity="30.0" effort="1.0"/>
+    <dynamics damping="1.0" friction="0.01"/>
   </joint>
-  <transmission name="wheel_back_transmission">
-    <type>transmission_interface/SimpleTransmission</type>
-    <joint name="wheel_back_joint">
-      <hardwareInterface>hardware_interface/EffortJointInterface</hardwareInterface>
-    </joint>
-    <actuator name="wheel_back_motor">
-      <hardwareInterface>hardware_interface/EffortJointInterface</hardwareInterface>
-      <mechanicalReduction>1</mechanicalReduction>
-    </actuator>
-  </transmission>
-  <gazebo reference="back_wheel_link">
-    <material>Gazebo/Black</material>
-    <selfCollide>false</selfCollide>
-    <gravity>true</gravity>
-    <collision name="back_wheel_link_collision">
-      <surface><friction>
-        <ode>
-          <mu>0.1</mu>
-          <mu2>15</mu2>
-          <fdir1>0 0 1</fdir1>
-        </ode></friction>
-      </surface>
+  <!-- LASER LINK AND JOINTS-->
+  <link name="laser_link">
+    <visual>
+      <origin xyz="0 0 0" rpy="0 0 0"/>
+      <geometry> <box size="0.05 0.05 0.08"/></geometry>
+      <material name="black"/>
+    </visual>
+    <collision>
+      <origin xyz="0 0 0" rpy="0 0 0"/>
+      <geometry> <box size="0.05 0.05 0.08"/></geometry>
     </collision>
-  </gazebo>
+    <inertial>
+      <origin xyz="0 0 0" rpy="0 0 0"/>
+      <mass value="0.1"/>
+      <xacro:box_inertia m="${0.1}" x="${0.05}" y="${0.05}" z="${0.08}"/>
+    </inertial>
+  </link>
+  <link name="laser_link_rear">
+    <visual>
+      <origin xyz="0 0 0" rpy="0 0 0"/>
+      <geometry> <box size="0.05 0.05 0.08"/></geometry>
+      <material name="black"/>
+    </visual>
+    <collision>
+      <origin xyz="0 0 0" rpy="0 0 0"/>
+      <geometry> <box size="0.05 0.05 0.08"/></geometry>
+    </collision>
+    <inertial>
+      <origin xyz="0 0 0" rpy="0 0 0"/>
+      <mass value="0.1"/>
+      <xacro:box_inertia m="${0.1}" x="${0.05}" y="${0.05}" z="${0.08}"/>
+    </inertial>
+  </link>
+  <joint name="laser_connect" type="fixed">
+    <origin xyz="0.17 0 0.14" />
+    <parent link="base_center"/>
+    <child link="laser_link"/>
+  </joint>
+  <joint name="rear_laser_connect" type="fixed">
+    <origin xyz="-0.2 0 0.14" rpy="0 0 ${PI}"/>
+    <parent link="base_center"/>
+    <child link="laser_link_rear"/>
+  </joint>
 </robot>
