Commit message: Add some files to simulate omnidirectional base in gazebo

File: catkin_ws/src/hardware/justina_description/urdf/justina_base_omni.xacro (robot description, xacro)
@@ -1,58 +1,174 @@
 <?xml version="1.0"?>
 <robot name="justina" xmlns:xacro="http://www.ros.org/wiki/xacro">
-  <!-- <xacro:include filename="$(find justina_description)/urdf/justina_base_rim.xacro"/> -->
+  <xacro:property name="base_radius" value="0.2"/>
+  <xacro:property name="base_height" value="0.2"/>
+  <xacro:property name="base_mass"   value="10.0"/>
+  <xacro:property name="wheel_radius" value="0.08"/>
+  <xacro:property name="wheel_width"  value="0.03"/>
+  <xacro:property name="wheel_mass"   value="0.5"/>
+  <xacro:property name="PI" value="3.14159265358979323846"/>
+  <xacro:include filename="$(find justina_description)/urdf/justina_base_rim.xacro"/>
   <link name="base_link"/>
-  <link name="base_box">
+  <link name="base_center">
     <inertial>
-      <mass value="0.07862944645"/>
-      <inertia
-	  ixx="0.00002035985530754"
-	  ixy="0"
-	  ixz="0"
-	  iyy="0.00002035985530754"
-	  iyz="0"
-	  izz="0.00003945961663220"/>
+      <origin xyz="0 0 0"/>
+      <mass value="${base_mass}"/>
+      <xacro:cylinder_inertia m="${base_mass}" r="${base_radius}" h="${base_height}"/>
     </inertial>
     <visual>
-      <geometry>
-        <cylinder radius="0.4" length="0.2"/>
-      </geometry>
-      <material name="base_material">
-	<color rgba="1 1 1 1"/>
-      </material>
+      <geometry><cylinder radius="${base_radius}" length="${base_height}"/></geometry>
+      <material name="base_material"><color rgba="0 0 1 1"/></material>
     </visual>
     <collision>
-      <geometry>
-        <cylinder radius="0.4" length="0.2"/>
-      </geometry>
+      <geometry><cylinder radius="${base_radius}" length="${base_height}"/></geometry>
     </collision>
   </link>
   <joint name="base_joint" type="fixed">
     <parent link="base_link" />
-    <child link="base_box" />
+    <child link="base_center" />
     <origin xyz="0 0 0.1905"/>
   </joint>
-  <!-- <xacro:rim_macro -->
-  <!--     name="left" -->
-  <!--     color="0.3 0 0" -->
-  <!--     xyz="-0.03464101615 0.02 0" -->
-  <!--     rpy="1.570796326794896 0 1.047197551196597" -->
-  <!--     /> -->
-  <!-- <xacro:rim_macro -->
-  <!--     name="back" -->
-  <!--     color="0 0.3 0" -->
-  <!--     xyz="0 -0.04 0" -->
-  <!--     rpy="1.570796326794896 0 3.141592653589793" -->
-  <!--     /> -->
-  <!-- <xacro:rim_macro -->
-  <!--     name="right" -->
-  <!--     color="0 0 0.3" -->
-  <!--     xyz="0.03464101615 0.02 0" -->
-  <!--     rpy="1.570796326794896 0 -1.047197551196597" -->
-  <!--     /> -->
-  <!-- <gazebo> -->
-  <!--   <plugin name="gazebo_ros_control" filename="libgazebo_ros_control.so"> -->
-  <!--     <robotNamespace>/justina</robotNamespace> -->
-  <!--   </plugin> -->
-  <!-- </gazebo> -->
+  <gazebo reference="base_center">
+    <material>Gazebo/Blue</material>
+    <selfCollide>false</selfCollide>
+    <gravity>true</gravity>
+  </gazebo>
+  <!-- LEFT WHEEL ACTUATOR-->
+  <link name="left_wheel_link">
+    <inertial>
+      <origin xyz="0 0 0"/>
+      <mass value="${wheel_mass}"/>
+      <xacro:cylinder_inertia m="${wheel_mass}" r="${wheel_radius}" h="${wheel_width}"/>
+    </inertial>
+    <visual>
+      <geometry><cylinder radius="${wheel_radius}" length="${wheel_width}"/></geometry>
+      <material name="wheel_material"><color rgba="0 0 0 1"/></material>
+    </visual>
+    <collision>
+      <geometry><cylinder radius="${wheel_radius}" length="${wheel_width}"/></geometry>
+    </collision>
+  </link>
+  <joint name="wheel_left_joint" type="continuous">
+    <parent link="base_center" />
+    <child link="left_wheel_link" />
+    <axis xyz="0 0 1"/>
+    <origin xyz="${(base_radius+0.03)*cos( PI/3)} ${(base_radius+0.03)*sin( PI/3)} -0.05" rpy="${PI/2} 0 ${ PI/3+PI/2}"/>
+    <limit velocity="30.0" effort="0.6"/>
+  </joint>
+  <transmission name="wheel_left_transmission">
+    <type>transmission_interface/SimpleTransmission</type>
+    <joint name="wheel_left_joint">
+      <hardwareInterface>hardware_interface/EffortJointInterface</hardwareInterface>
+    </joint>
+    <actuator name="wheel_left_motor">
+      <hardwareInterface>hardware_interface/EffortJointInterface</hardwareInterface>
+      <mechanicalReduction>1</mechanicalReduction>
+    </actuator>
+  </transmission>
+  <gazebo reference="left_wheel_link">
+    <material>Gazebo/Black</material>
+    <selfCollide>false</selfCollide>
+    <gravity>true</gravity>
+    <collision name="left_wheel_link_collision">
+      <surface><friction>
+        <ode>
+          <mu>0.1</mu>
+          <mu2>15</mu2>
+          <fdir1>0 0 1</fdir1>
+        </ode></friction>
+      </surface>
+    </collision>
+  </gazebo>
+  <!-- RIGHT WHEEL ACTUATOR-->
+  <link name="right_wheel_link">
+    <inertial>
+      <origin xyz="0 0 0"/>
+      <mass value="${wheel_mass}"/>
+      <xacro:cylinder_inertia m="${wheel_mass}" r="${wheel_radius}" h="${wheel_width}"/>
+    </inertial>
+    <visual>
+      <geometry><cylinder radius="${wheel_radius}" length="${wheel_width}"/></geometry>
+      <material name="wheel_material"><color rgba="0 0 0 1"/></material>
+    </visual>
+    <collision>
+      <geometry><cylinder radius="${wheel_radius}" length="${wheel_width}"/></geometry>
+    </collision>
+  </link>
+  <joint name="wheel_right_joint" type="continuous">
+    <parent link="base_center" />
+    <child link="right_wheel_link" />
+    <axis xyz="0 0 1"/>
+    <origin xyz="${(base_radius+0.03)*cos(-PI/3)} ${(base_radius+0.03)*sin(-PI/3)} -0.05" rpy="${PI/2} 0 ${-PI/3+PI/2}"/>
+    <limit velocity="30.0" effort="0.6"/>
+  </joint>
+  <transmission name="wheel_right_transmission">
+    <type>transmission_interface/SimpleTransmission</type>
+    <joint name="wheel_right_joint">
+      <hardwareInterface>hardware_interface/EffortJointInterface</hardwareInterface>
+    </joint>
+    <actuator name="wheel_right_motor">
+      <hardwareInterface>hardware_interface/EffortJointInterface</hardwareInterface>
+      <mechanicalReduction>1</mechanicalReduction>
+    </actuator>
+  </transmission>
+  <gazebo reference="right_wheel_link">
+    <material>Gazebo/Black</material>
+    <selfCollide>false</selfCollide>
+    <gravity>true</gravity>
+    <collision name="right_wheel_link_collision">
+      <surface><friction>
+        <ode>
+          <mu>0.1</mu>
+          <mu2>15</mu2>
+          <fdir1>0 0 1</fdir1>
+        </ode></friction>
+      </surface>
+    </collision>
+  </gazebo>
+  <!-- BACK WHEEL ACTUATOR-->
+  <link name="back_wheel_link">
+    <inertial>
+      <origin xyz="0 0 0"/>
+      <mass value="${wheel_mass}"/>
+      <xacro:cylinder_inertia m="${wheel_mass}" r="${wheel_radius}" h="${wheel_width}"/>
+    </inertial>
+    <visual>
+      <geometry><cylinder radius="${wheel_radius}" length="${wheel_width}"/></geometry>
+      <material name="wheel_material"><color rgba="0 0 0 1"/></material>
+    </visual>
+    <collision>
+      <geometry><cylinder radius="${wheel_radius}" length="${wheel_width}"/></geometry>
+    </collision>
+  </link>
+  <joint name="wheel_back_joint" type="continuous">
+    <parent link="base_center" />
+    <child link="back_wheel_link" />
+    <axis xyz="0 0 1"/>
+    <origin xyz="${(base_radius+0.03)*cos(PI)} ${(base_radius+0.03)*sin(PI)} -0.05" rpy="${PI/2} 0 ${PI+PI/2}"/>
+    <limit velocity="30.0" effort="0.6"/>
+  </joint>
+  <transmission name="wheel_back_transmission">
+    <type>transmission_interface/SimpleTransmission</type>
+    <joint name="wheel_back_joint">
+      <hardwareInterface>hardware_interface/EffortJointInterface</hardwareInterface>
+    </joint>
+    <actuator name="wheel_back_motor">
+      <hardwareInterface>hardware_interface/EffortJointInterface</hardwareInterface>
+      <mechanicalReduction>1</mechanicalReduction>
+    </actuator>
+  </transmission>
+  <gazebo reference="back_wheel_link">
+    <material>Gazebo/Black</material>
+    <selfCollide>false</selfCollide>
+    <gravity>true</gravity>
+    <collision name="back_wheel_link_collision">
+      <surface><friction>
+        <ode>
+          <mu>0.1</mu>
+          <mu2>15</mu2>
+          <fdir1>0 0 1</fdir1>
+        </ode></friction>
+      </surface>
+    </collision>
+  </gazebo>
 </robot>

File: catkin_ws/src/hardware/justina_description/urdf/justina_base_rim.xacro (robot description, xacro)
@@ -2,20 +2,17 @@
 <robot xmlns:xacro="http://www.ros.org/wiki/xacro">
   <xacro:include filename="$(find justina_description)/urdf/justina_base_roller.xacro"/>
+  <xacro:property name="rim_radius" value="0.08"/>
+  <xacro:property name="rim_width" value="0.0221"/>
+  <xacro:property name="PI" value="3.14159265358979323846"/>
   <xacro:macro name="rim_macro" params="name color xyz rpy"	>
     <link name="rim_${name}_link">
       <inertial>
-	<origin xyz="0 0 -0.000343"/>
-	<mass value="0.0835758"/>
-	<inertia
-	    ixx="6.63684e-06"
-	    ixy="0"
-	    ixz="0"
-	    iyy="6.63684e-06"
-	    iyz="0"
-	    izz="9.40333e-06"/>
+        <origin xyz="0 0 0"/>
+        <mass value="0.1"/>
+        <xacro:cylinder_inertia m="0.1" r="${rim_radius}" h="${rim_width}"/>
       </inertial>
       <visual>
 	<geometry>
-	  <mesh filename="package://justina_description/stl/justina_base_rim.stl"/>
+	  <mesh filename="package://justina_description/stl/justina_base_rim.stl" scale="5 5 2"/>
 	</geometry>
 	<material name="rim_${name}_material">
@@ -25,72 +22,37 @@
       <collision>
 	<geometry>
-	  <mesh filename="package://justina_description/stl/justina_base_rim.stl"/>
+	  <mesh filename="package://justina_description/stl/justina_base_rim.stl" scale ="5 5 2"/>
 	</geometry>
       </collision>
     </link>
-    <joint name="rim_${name}_joint" type="continuous">
-      <parent link="base_link" />
+    <joint name="wheel_${name}_joint" type="continuous">
+      <parent link="base_center" />
       <child link="rim_${name}_link" />
       <axis xyz="0 0 1"/>
       <origin xyz="${xyz}" rpy="${rpy}"/>
     </joint>
-    <xacro:roller_macro
-	parent="${name}"
-	name="e"
-	xyz="0.01355 0 0.0055"
-	rpy="-1.570796326794896 0 0"
-	/>
-    <xacro:roller_macro
-	parent="${name}"
-	name="ne"
-	xyz="0.00958129689 0.00958129689 -0.0055"
-	rpy="-1.570796326794896 0 0.7853981633974483"
-	/>
-    <xacro:roller_macro
-	parent="${name}"
-	name="n"
-	xyz="0 0.01355 0.0055"
-	rpy="-1.570796326794896 0 1.570796326794896"
-	/>
-    <xacro:roller_macro
-	parent="${name}"
-	name="nw"
-	xyz="-0.00958129689 0.00958129689 -0.0055"
-	rpy="-1.570796326794896 0 2.356194490192345"
-	/>
-    <xacro:roller_macro
-	parent="${name}"
-	name="w"
-	xyz="-0.01355 0 0.0055"
-	rpy="-1.570796326794896 0 3.141592653589793"
-	/>
-    <xacro:roller_macro
-	parent="${name}"
-	name="sw"
-	xyz="-0.00958129689 -0.00958129689 -0.0055"
-	rpy="-1.570796326794896 0 -2.356194490192345"
-	/>
-    <xacro:roller_macro
-	parent="${name}"
-	name="s"
-	xyz="0 -0.01355 0.0055"
-	rpy="-1.570796326794896 0 -1.570796326794896"
-	/>
-    <xacro:roller_macro
-	parent="${name}"
-	name="se"
-	xyz="0.00958129689 -0.00958129689 -0.0055"
-	rpy="-1.570796326794896 0 -0.7853981633974483"
-	/>
+    <xacro:roller_macro parent="${name}" name="e"  xyz="${ rim_radius}       0        ${ rim_width/2}" rpy="${-PI/2} 0 0"/>
+    <xacro:roller_macro	parent="${name}" name="n"  xyz="          0    ${ rim_radius} ${ rim_width/2}" rpy="${-PI/2} 0 ${PI/2}"/>
+    <xacro:roller_macro parent="${name}" name="w"  xyz="${-rim_radius}       0        ${ rim_width/2}" rpy="${-PI/2} 0 ${PI}"/>
+    <xacro:roller_macro	parent="${name}" name="s"  xyz="          0    ${-rim_radius} ${ rim_width/2}" rpy="${-PI/2} 0 ${3*PI/2}"/>
+    <xacro:roller_macro parent="${name}" name="ne" xyz="${ rim_radius/sqrt(2)} ${ rim_radius/sqrt(2)} ${-rim_width/2}" rpy="${-PI/2} 0 ${PI/4}"/>
+    <xacro:roller_macro parent="${name}" name="nw" xyz="${-rim_radius/sqrt(2)} ${ rim_radius/sqrt(2)} ${-rim_width/2}" rpy="${-PI/2} 0 ${3*PI/4}"/>
+    <xacro:roller_macro parent="${name}" name="sw" xyz="${-rim_radius/sqrt(2)} ${-rim_radius/sqrt(2)} ${-rim_width/2}" rpy="${-PI/2} 0 ${5*PI/4}"/>
+    <xacro:roller_macro parent="${name}" name="se" xyz="${ rim_radius/sqrt(2)} ${-rim_radius/sqrt(2)} ${-rim_width/2}" rpy="${-PI/2} 0 ${7*PI/4}"/>
     <transmission name="rim_${name}_transmission">
       <type>transmission_interface/SimpleTransmission</type>
-      <joint name="rim_${name}_joint">
-	<hardwareInterface>EffortJointInterface</hardwareInterface>
+      <joint name="wheel_${name}_joint">
+	<hardwareInterface>hardware_interface/VelocityJointInterface</hardwareInterface>
       </joint>
       <actuator name="rim_${name}_motor">
-	<hardwareInterface>EffortJointInterface</hardwareInterface>
+	<hardwareInterface>hardware_interface/VelocityJointInterface</hardwareInterface>
 	<mechanicalReduction>1</mechanicalReduction>
       </actuator>
     </transmission>
+    <gazebo reference="rim_${name}_link">
+      <material>Gazebo/Gray</material>
+      <selfCollide>false</selfCollide>
+      <gravity>true</gravity>
+    </gazebo>
   </xacro:macro>
 </robot>

File: catkin_ws/src/hardware/justina_description/urdf/justina_base_roller.xacro (robot description, xacro)
@@ -1,20 +1,17 @@
 <?xml version="1.0" ?>
 <robot xmlns:xacro="http://www.ros.org/wiki/xacro">
+  <macro name="cylinder_inertia" params="m r h">
+    <inertia  ixx="${m*(3*r*r+h*h)/12}" ixy = "0" ixz = "0" iyy="${m*(3*r*r+h*h)/12}" iyz = "0" izz="${m*r*r/2}"/>
+  </macro>
   <xacro:macro name="roller_macro" params="parent name xyz rpy">
     <link name="roller_${name}_rim_${parent}_link">
       <inertial>
-        <mass value="0.00113845"/>
-	<inertia
-	    ixx="2.53776e-08"
-	    ixy="0"
-	    ixz="0"
-	    iyy="2.53776e-08"
-	    iyz="0"
-	    izz="1.47666e-08"
-	    />
+        <origin xyz="0 0 0"/>
+        <mass value="0.02"/>
+        <xacro:cylinder_inertia m="0.02" r="0.005" h="0.03"/>
       </inertial>
       <visual>
         <geometry>
-          <mesh filename="package://justina_description/stl/justina_base_roller.stl"/>
+          <mesh filename="package://justina_description/stl/justina_base_roller.stl" scale="2 2 5"/>
 	</geometry>
 	<material name="roller_material">
@@ -24,5 +21,5 @@
       <collision>
 	<geometry>
-	  <mesh filename="package://justina_description/stl/justina_base_roller.stl"/>
+	  <mesh filename="package://justina_description/stl/justina_base_roller.stl" scale="2 2 5"/>
 	</geometry>
       </collision>
@@ -34,4 +31,9 @@
       <origin xyz="${xyz}" rpy="${rpy}"/>
     </joint>
+    <gazebo reference="roller_${name}_rim_${parent}_link">
+      <material>Gazebo/Black</material>
+      <selfCollide>false</selfCollide>
+      <gravity>true</gravity>
+    </gazebo>
   </xacro:macro>
 </robot>

Commit message: Rename justina controller files Correct omni base gazebo control for better speed control and correct odometry Modify launch files Add buttons to gui for lateral moving. Still not working

File: catkin_ws/src/hardware/justina_description/urdf/justina_base_omni.xacro (robot description, xacro)
@@ -44,5 +44,5 @@
     <parent link="base_link" />
     <child link="base_center" />
-    <origin xyz="0 0 0.1905"/>
+    <origin xyz="0 0 0.13"/>
   </joint>
   <joint name="base_torso_support_joint" type="fixed">
@@ -71,6 +71,6 @@
     <axis xyz="0 0 1"/>
     <origin xyz="${(base_radius+0.03)*cos( PI/3)} ${(base_radius+0.03)*sin( PI/3)} -0.05" rpy="${PI/2} 0 ${ PI/3+PI/2}"/>
-    <limit velocity="30.0" effort="1.0"/>
-    <dynamics damping="1.0" friction="0.01"/>
+    <limit velocity="30.0" effort="5.0"/>
+    <dynamics damping="0.5" friction="0.01"/>
   </joint>
   <!-- RIGHT WHEEL ACTUATOR-->
@@ -94,6 +94,6 @@
     <axis xyz="0 0 1"/>
     <origin xyz="${(base_radius+0.03)*cos(-PI/3)} ${(base_radius+0.03)*sin(-PI/3)} -0.05" rpy="${PI/2} 0 ${-PI/3+PI/2}"/>
-    <limit velocity="30.0" effort="1.0"/>
-    <dynamics damping="1.0" friction="0.01"/>
+    <limit velocity="30.0" effort="5.0"/>
+    <dynamics damping="0.5" friction="0.01"/>
   </joint>
   <!-- BACK WHEEL ACTUATOR-->
@@ -117,6 +117,6 @@
     <axis xyz="0 0 1"/>
     <origin xyz="${(base_radius+0.03)*cos(PI)} ${(base_radius+0.03)*sin(PI)} -0.05" rpy="${PI/2} 0 ${PI+PI/2}"/>
-    <limit velocity="30.0" effort="1.0"/>
-    <dynamics damping="1.0" friction="0.01"/>
+    <limit velocity="30.0" effort="5.0"/>
+    <dynamics damping="0.5" friction="0.01"/>
   </joint>
   <!-- LASER LINK AND JOINTS-->
